Commit message: Adding project files

File: catkin_ws/src/my_robot/urdf/my_robot.xacro (robot description, xacro)
@@ -30,8 +30,8 @@
     <axis xyz="0 1 0" rpy="0 0 0"/>
   </joint>
-  <gazebo reference="camera">
-  <material>Gazebo/Yellow</material>
-  </gazebo>
-  <link name="camera">
+  <gazebo reference="camera_link">
+  <material>Gazebo/Black</material>
+  </gazebo>
+  <link name="camera_link">
    <visual>
      <origin xyz="0 0 0" rpy="0 0 0" />
@@ -58,8 +58,15 @@
  <joint type="fixed" name="camera_joint">
     <origin xyz="0.2 0 0" rpy="0 0 0"/>
-    <child link="camera"/>
-    <parent link="chassis"/>
-    <axis xyz="0 1 0" rpy="0 0 0"/>
-  </joint>
+    <child link="camera_link"/>
+    <parent link="chassis"/>
+    <axis xyz="0 1 0" rpy="0 0 0"/>
+  </joint>
+   <joint name="camera_optical_joint" type="fixed">
+    <origin xyz="0 0 0" rpy="-1.5707 0 -1.5707"/>
+    <parent link="camera_link"/>
+    <child link="camera_link_optical"/>
+  </joint>
+  <link name="camera_link_optical">
+  </link>
   <gazebo reference="left_whell">
    <material>Gazebo/Black</material>
@@ -96,5 +103,8 @@
     <dynamics damping="1.0" friction="1.0"/>
   </joint>
-  <gazebo reference="right_whell">
+  <gazebo reference="right_wheel">
+   <material>Gazebo/Black</material>
+  </gazebo>
+  <gazebo reference="left_wheel">
    <material>Gazebo/Black</material>
   </gazebo>

Commit message: Organized structure
Removed bugs, organized the xacro file, changed "robot_footprint" to "base_footprint". Mapping now works!

File: catkin_ws/src/my_robot/urdf/my_robot.xacro (robot description, xacro)
@@ -1,4 +1,46 @@
 <?xml version='1.0'?>
 <robot name="my_robot" xmlns:xacro="http://www.ros.org/wiki/xacro">
+<xacro:include filename="$(find my_robot)/urdf/my_robot.gazebo" />
+<link name="base_footprint"></link>
+<!-- Joints-->
+  <joint type="continuous" name="right_wheel_hinge">
+    <origin xyz="0 -0.15 0" rpy="0 0 0"/>
+    <child link="right_wheel"/>
+    <parent link="chassis"/>
+    <axis xyz="0 1 0" rpy="0 0 0"/>
+    <limit effort="10000" velocity="1000"/>
+    <dynamics damping="1.0" friction="1.0"/>
+  </joint>
+  <joint name="base_footprint_joint" type="fixed">
+    <origin xyz="0 0 0" rpy="0 0 0" />
+    <parent link="base_footprint"/>
+    <child link="chassis" />
+  </joint>
+  <joint type="fixed" name="hokuyo_joint">
+    <origin xyz="0.15 0 .1" rpy="0 0 0"/>
+    <child link="hokuyo"/>
+    <parent link="chassis"/>
+    <axis xyz="0 1 0" rpy="0 0 0"/>
+  </joint>
+  <joint type="continuous" name="left_wheel_hinge">
+    <origin xyz="0 0.15 0" rpy="0 0 0"/>
+    <child link="left_wheel"/>
+    <parent link="chassis"/>
+    <axis xyz="0 1 0" rpy="0 0 0"/>
+    <limit effort="10000" velocity="1000"/>
+    <dynamics damping="1.0" friction="1.0"/>
+  </joint>
+  <joint type="fixed" name="camera_joint">
+    <origin xyz="0.2 0 0" rpy="0 0 0"/>
+    <child link="camera_link"/>
+    <parent link="chassis"/>
+    <axis xyz="0 1 0" rpy="0 0 0"/>
+  </joint>
+   <joint name="camera_optical_joint" type="fixed">
+    <origin xyz="0 0 0" rpy="-1.5707 0 -1.5707"/>
+    <parent link="camera_link"/>
+    <child link="camera_link_optical"/>
+  </joint>
+<!-- Links -->
 <link name="hokuyo">
    <visual>
@@ -24,14 +66,5 @@
    </inertial>
  </link>
- <joint type="fixed" name="hokuyo_joint">
-    <origin xyz="0.15 0 .1" rpy="0 0 0"/>
-    <child link="hokuyo"/>
-    <parent link="chassis"/>
-    <axis xyz="0 1 0" rpy="0 0 0"/>
-  </joint>
-  <gazebo reference="camera_link">
-  <material>Gazebo/Black</material>
-  </gazebo>
-  <link name="camera_link">
+ <link name="camera_link">
    <visual>
      <origin xyz="0 0 0" rpy="0 0 0" />
@@ -56,20 +89,4 @@
    </inertial>
  </link>
- <joint type="fixed" name="camera_joint">
-    <origin xyz="0.2 0 0" rpy="0 0 0"/>
-    <child link="camera_link"/>
-    <parent link="chassis"/>
-    <axis xyz="0 1 0" rpy="0 0 0"/>
-  </joint>
-   <joint name="camera_optical_joint" type="fixed">
-    <origin xyz="0 0 0" rpy="-1.5707 0 -1.5707"/>
-    <parent link="camera_link"/>
-    <child link="camera_link_optical"/>
-  </joint>
-  <link name="camera_link_optical">
-  </link>
-  <gazebo reference="left_whell">
-   <material>Gazebo/Black</material>
-  </gazebo>
   <link name="left_wheel">
     <inertial>
@@ -95,18 +112,4 @@
     </visual>
   </link>
-  <joint type="continuous" name="left_wheel_hinge">
-    <origin xyz="0 0.15 0" rpy="0 0 0"/>
-    <child link="left_wheel"/>
-    <parent link="chassis"/>
-    <axis xyz="0 1 0" rpy="0 0 0"/>
-    <limit effort="10000" velocity="1000"/>
-    <dynamics damping="1.0" friction="1.0"/>
-  </joint>
-  <gazebo reference="right_wheel">
-   <material>Gazebo/Black</material>
-  </gazebo>
-  <gazebo reference="left_wheel">
-   <material>Gazebo/Black</material>
-  </gazebo>
   <link name="right_wheel">
     <inertial>
@@ -132,22 +135,4 @@
     </visual>
   </link>
-  <joint type="continuous" name="right_wheel_hinge">
-    <origin xyz="0 -0.15 0" rpy="0 0 0"/>
-    <child link="right_wheel"/>
-    <parent link="chassis"/>
-    <axis xyz="0 1 0" rpy="0 0 0"/>
-    <limit effort="10000" velocity="1000"/>
-    <dynamics damping="1.0" friction="1.0"/>
-  </joint>
-  <xacro:include filename="$(find my_robot)/urdf/my_robot.gazebo" />
-  <link name="robot_footprint"></link>
-  <joint name="robot_footprint_joint" type="fixed">
-    <origin xyz="0 0 0" rpy="0 0 0" />
-    <parent link="robot_footprint"/>
-    <child link="chassis" />
-  </joint>
-<gazebo reference="chassis">
-   <material>Gazebo/Blue</material>
-  </gazebo>
   <link name='chassis'>
     <pose>0 0 0.1 0 0 0</pose>
@@ -197,4 +182,20 @@
       </geometry>
     </visual>
+ </link>
+<link name="camera_link_optical">
   </link>
+<!-- Colors -->
+  <gazebo reference="chassis">
+   <material>Gazebo/Blue</material>
+  </gazebo>
+  <gazebo reference="right_wheel">
+   <material>Gazebo/Black</material>
+  </gazebo>
+  <gazebo reference="left_wheel">
+   <material>Gazebo/Black</material>
+  </gazebo>
+  <gazebo reference="camera_link">
+   <material>Gazebo/Black</material>
+  </gazebo>
+<!-- END -->
 </robot>
